File: pcb/metronome.brd (EAGLE design)
At the start: 100 x 80 mm, 81 parts, among them J1 FCI_CORTEX_SWD_CONNECTOR, J2 POWER_JACKPTH, J3 MINI_USB_B, J5 MINI_USB_B, U1 ATSAMD4S2BA-AU

Commit message: finished board design
Parts:
- removed R10, R11, R8, R9: 0Ohm, adafruit:R0402
- added AD1, VREF: TPSQTP13SQ, testpad:TP13SQ
- added C35, C38, C42: 1uF, adafruit:C0402
- added C36, C37, C39, C43: 10uF, john_mamish_passives_library:PANASONIC_EEEHB100AR
- added C40, C41: .33uF, adafruit:C0402
- added C44: 4.7uF, adafruit:C0603
- added D2, D3, D4: BLUE, john_mamish_assorted_analog_library:D0603
- added JP1: (no value), pinhead:1X03
- added R21, R22, R23, R25: 22Ohm, adafruit:R0402
- added R24, R26, R27, R30, R32, R33, R34, R35, R36, R37, R38, R39, R40, R41, R42, R43, R44: 10kOhm, adafruit:R0402
- added R28, R29: 20kOhm, adafruit:R0402
- added R31: 220kOhm, adafruit:R0402
- added R45, R46, R47: 100Ohm, adafruit:R0402
- added SB1, SB2, SB3, SB4, SB5: SB_1MM, john_mamish_passives_library:SB_1MM
- added SPK2+, SPK2-, SPKR0, SPRK1: TPSQTP20SQ, testpad:TP20SQ
- added SW1, SW2, SW3, SW4, SW5, SW6, SW7, SW8: (no value), john_mamish_passives_library:FSMJSMA
- added U$10: MAXIM_MAX_98307, john_mamish_assorted_analog_library:MAXIM_16_TQFN_T1633-5
- added U$11: BOURNS_PEC16-4215F-S0024, john_mamish_passives_library:BOURNS_PEC16-4XXXF-SXXXX
- added U$6, U$8: 330uF, john_mamish_passives_library:PANASONIC_EEEFT0JXXX
- added U$9: TI_PCM1789, john_mamish_dacs_and_adcs:TI_PW_TSSOP_24
- C1: value (none) -> 330nF
- moved TP_+3V33 447.6 mm to (42.1, 78.4), turned to 180 degrees
- moved TP_GND2 435.3 mm to (98.1, 78.0), turned to 90 degrees
- moved TP_+3V32 429.1 mm to (98.1, 54.0), turned to 90 degrees
- moved TP_GND3 427.7 mm to (10.0, 78.4), turned to 180 degrees
- moved TP_URXDO 422.7 mm to (22.6, 41.9), turned to 180 degrees
- moved TP_UTXD0 421.6 mm to (22.6, 45.2), turned to 180 degrees
- moved R17 386.6 mm to (35.4, 72.0), turned to 270 degrees
- moved R20 386.0 mm to (44.4, 52.2), turned to 180 degrees
- moved TP_+5V0 381.8 mm to (76.8, 1.60)
- moved R19 380.0 mm to (44.4, 51.1)
- moved R18 372.9 mm to (47.8, 48.5)
- moved TP_+3V31 360.3 mm to (18.0, 1.70)
- moved TP_+3V30 355.7 mm to (14.9, 1.70)
- moved C34 343.6 mm to (43.6, 70.1), turned to 90 degrees
- moved R16 343.2 mm to (9.50, 35.5), turned to 90 degrees
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Connections:
- net N$2 renamed SERIAL_USB-
- net SERIAL_ renamed SERIAL_USB+
- removed net CPLD_JTAG_NRST: J4.15
- removed net CPLD_JTAG_NTRST: J4.3
- removed net I2S_LR_SELECT: U$2.11, U1.P$20
- removed net N$12: R9.2, U$1.P$41
- removed net N$14: R8.2, U$1.P$40
- removed net PCM_1774_SYSCLK: U$2.9, U1.P$59
- new net CPLD_PROGRAMN: R41.1, SB5.P$1, SW8.P$1, SW8.P$2, U$1.P$81
- new net ENC_A: R42.1, U$1.P$1, U$11.A
- new net ENC_B: R43.1, U$1.P$2, U$11.B
- new net ENC_SWITCH: R44.2, U$1.P$24, U$11.E
- new net I2S_DATA_MCU: R21.2, U1.P$9
- new net I2S_LRCK: R23.1, U$2.11, U$9.P$1
- new net I2S_LR_SELECT_MCU: R23.2, U1.P$20
- new net LED_1: R45.1, U1.P$6
- new net LED_2: R46.1, U1.P$5
- new net LED_3: R47.1, U1.P$4
- new net MAX98307_PUMP_VSS: C43.POS, U$10.P$14, U$10.P$7
- new net MAX98307_VCC: JP1.2, U$10.P$1, U$10.P$13, U$10.P$3
- new net N$2: SB2.P$2, U$1.P$41
- new net N$25: SB1.P$2, U$1.P$40
- new net N$26: U$2.15, U$6.POS
- new net N$27: U$2.14, U$8.POS
- new net N$28: SPRK1.TP, U$8.NEG
- new net N$29: R22.2, U1.P$19
- new net N$3: SPKR0.TP, U$6.NEG
- new net N$30: R25.1, U1.P$59
- new net N$31: C41.1, U$9.P$14
- new net N$32: C40.1, U$9.P$13
- new net N$33: C41.2, R27.2
- new net N$34: C40.2, R26.2
- new net N$35: R26.1, R28.1, U$10.P$11
- new net N$36: R27.1, R29.1, U$10.P$10
- new net N$37: R28.2, U$10.P$12
- new net N$38: C39.POS, U$9.P$9
- new net N$39: R29.2, U$10.P$9
- new net N$42: R31.1, U$9.P$20
- new net N$43: R32.1, U$9.P$24
- new net N$44: D2.AN, R45.2
- new net N$45: D3.AN, R46.2
- new net N$46: SPK2+.TP, U$10.P$4
- new net N$47: SPK2-.TP, U$10.P$5
- new net N$48: D4.AN, R47.2
- new net N$49: J4.15, SB5.P$2
- new net N$52: R33.1, U$9.P$23
- new net N$53: C44.2, U$10.P$15
- new net N$54: C44.1, U$10.P$16
- new net N$7: U1.P$1, VREF.TP
- new net N$8: AD1.TP, U1.P$10
- new net PCM1789_MUTE: R30.1, U$9.P$17
- new net PCM_17XX_SYSCLK: R25.2, U$2.9, U$9.P$5
- new net SW_1: R34.2, SW1.P$3, SW1.P$4, U$1.P$14
- new net SW_2: R35.2, SW2.P$3, SW2.P$4, U$1.P$15
- new net SW_3: R36.2, SW3.P$3, SW3.P$4, U$1.P$16
- new net SW_4: R37.2, SW4.P$3, SW4.P$4, U$1.P$17
- new net SW_5: R38.2, SW5.P$3, SW5.P$4, U$1.P$18
- new net SW_6: R39.2, SW6.P$3, SW6.P$4, U$1.P$19
- net !DISP_RESET!: now also R40.1, U1.P$31
- net +3V3: now also C35.1, C36.POS, JP1.3, R24.2, R30.2, R40.2, R41.2, R42.2, R43.2, SW1.P$1, SW1.P$2, SW2.P$1, SW2.P$2, SW3.P$1, SW3.P$2, SW4.P$1, SW4.P$2, SW5.P$1, SW5.P$2, SW6.P$1, SW6.P$2, U$1.P$73, U$11.D, U$9.P$6
- net +5V0: now also C37.POS, C38.1, C42.1, JP1.1, U$9.P$16, U$9.P$8
- net DISP_CHIP_SELECT: now also U$1.P$96; no longer U$1.P$78
- net DISP_DB13: now also U$1.P$74; no longer U$1.P$73
- net DISP_DB14: now also U$1.P$75; no longer U$1.P$74
- net DISP_DB15: now also U$1.P$78; no longer U$1.P$75
- net DISP_SPI_CS: now also SB4.P$1; no longer R11.1
- net DISP_SPI_MISO: now also SB1.P$1; no longer R8.1
- net DISP_SPI_MOSI: now also SB3.P$1; no longer R10.1
- net DISP_SPI_SPCK: now also SB2.P$1; no longer R9.1
- net GND: now also C35.2, C36.NEG, C37.NEG, C38.2, C39.NEG, C42.2, C43.NEG, D2.CATH, D3.CATH, D4.CATH, R31.2, R32.2, R33.2, R34.1, R35.1, R36.1, R37.1, R38.1, R39.1, R44.1, SW7.P$1, SW7.P$2, SW8.P$3, SW8.P$4, U$10.P$17, U$10.P$2, U$10.P$6, U$11.C, U$9.P$10, U$9.P$15, U$9.P$7
- net I2S_BCK: now also R22.1, U$9.P$2; no longer U1.P$19
- net I2S_DATA: now also R21.1, U$9.P$3; no longer U1.P$9
- net N$10: now also SB4.P$2; no longer R11.2
- net N$11: now also SB3.P$2; no longer R10.2
- net SAM4S_NRST: now also R24.1, SW7.P$3, SW7.P$4, U$9.P$4
- net TWCK0: now also U$1.P$86, U$9.P$22
- net TWD0: now also U$1.P$85, U$9.P$21
- net VBUS_DETECT: now also U1.P$38
Routing:
- net +3V3: track 22.6 -> 680.1 mm, vias 0 -> 35
- net ENC_SWITCH: track 0.00 -> 117.3 mm, vias 0 -> 4
- net ENC_B: track 0.00 -> 112.6 mm, vias 0 -> 3
- net ENC_A: track 0.00 -> 107.5 mm, vias 0 -> 3
- net +5V0: track 0.00 -> 101.1 mm, vias 0 -> 3
- net SW_6: track 0.00 -> 99.2 mm, vias 0 -> 2
- net SAM4S_NRST: track 0.00 -> 98.1 mm, vias 0 -> 8
- net TWD0: track 0.00 -> 90.8 mm, vias 0 -> 5
- net SW_5: track 0.00 -> 90.1 mm, vias 0 -> 2
- net TWCK0: track 0.00 -> 83.3 mm, vias 0 -> 5
- net SW_4: track 0.00 -> 79.2 mm, vias 0 -> 2
- net SW_1: track 0.00 -> 73.7 mm, vias 0 -> 2
- net SW_3: track 0.00 -> 66.9 mm, vias 0 -> 2
- net SW_2: track 0.00 -> 66.3 mm, vias 0 -> 2
- net !DISP_RESET!: track 0.00 -> 52.9 mm, vias 0 -> 2
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Other:
- board text added: "3.3v"
- board text added: "5.0v"
- board text added: "Connect JTAG to \PROGRAMn"
- board text added: "SAM4S reset"
- board text added: "Serial port"
- board text added: "USB"
