File: pcb/metronome.sch (EAGLE design)
At the start: 81 parts, among them J1 FCI_CORTEX_SWD_CONNECTOR, J2 POWER_JACKPTH, J3 MINI_USB_B, J5 MINI_USB_B, U1 ATSAMD4S2BA-AU

Commit message: finished board design
Parts:
- removed R10, R11, R8, R9: 0Ohm, adafruit:R-US_R0402
- added AD1, VREF: TPSQTP13SQ, testpad:TPSQTP13SQ
- added C35, C38, C42: 1uF, adafruit:C-USC0402
- added C36, C37, C39, C43: 10uF, john_mamish_passives_library:PANASONIC_HB1C100AR
- added C40, C41: .33uF, adafruit:C-USC0402
- added C44: 4.7uF, adafruit:C-USC0603
- added D2, D3, D4: BLUE, john_mamish_assorted_analog_library:LED0603
- added JP1: (no value), pinhead:PINHD-1X3
- added R21, R22, R23, R25: 22Ohm, adafruit:R-US_R0402
- added R24, R26, R27, R30, R32, R33, R34, R35, R36, R37, R38, R39, R40, R41, R42, R43, R44: 10kOhm, adafruit:R-US_R0402
- added R28, R29: 20kOhm, adafruit:R-US_R0402
- added R31: 220kOhm, adafruit:R-US_R0402
- added R45, R46, R47: 100Ohm, adafruit:R-US_R0402
- added SB1, SB2, SB3, SB4, SB5: SB_1MM, john_mamish_passives_library:SB_1MM
- added SPK2+, SPK2-, SPKR0, SPRK1: TPSQTP20SQ, testpad:TPSQTP20SQ
- added SW1, SW2, SW3, SW4, SW5, SW6, SW7, SW8: (no value), john_mamish_passives_library:FSMJSMA
- added U$10: MAXIM_MAX_98307, john_mamish_assorted_analog_library:MAXIM_MAX_98307
- added U$11: BOURNS_PEC16-4215F-S0024, john_mamish_passives_library:BOURNS_PEC16-4215F-S0024
- added U$6, U$8: 330uF, john_mamish_passives_library:PANASONIC_EEEFT0JXXX
- added U$9: TI_PCM1789, john_mamish_dacs_and_adcs:TI_PCM1789
- C1: value (none) -> 330nF
Connections:
- net N$2 renamed SERIAL_USB-
- net SERIAL_ renamed SERIAL_USB+
- removed net CPLD_JTAG_NRST: J4.15
- removed net CPLD_JTAG_NTRST: J4.3
- removed net I2S_LR_SELECT: U$2.LRCK, U1.PA15/PGMD3
- removed net N$12: R9.2, U$1.PB12B
- removed net N$14: R8.2, U$1.PB12A
- removed net PCM_1774_SYSCLK: U$2.SCKI, U1.PB13/DAC0
- new net CPLD_PROGRAMN: R41.1, SB5.P$1, SW8.P$1, SW8.P$2, U$1.PT10D/PROGRAMN
- new net ENC_A: R42.1, U$1.PL2A, U$11.A
- new net ENC_B: R43.1, U$1.PL2B, U$11.B
- new net ENC_SWITCH: R44.2, U$1.PL7C, U$11.E
- new net I2S_DATA_MCU: R21.2, U1.PA17/PGMD5/AD0
- new net I2S_LRCK: R23.1, U$2.LRCK, U$9.LRCK
- new net I2S_LR_SELECT_MCU: R23.2, U1.PA15/PGMD3
- new net LED_1: R45.1, U1.PB3/AD7
- new net LED_2: R46.1, U1.PB2/AD6
- new net LED_3: R47.1, U1.PB1/AD5
- new net MAX98307_PUMP_VSS: C43.POS, U$10.PVSS, U$10.SVSS
- new net MAX98307_VCC: JP1.2, U$10.!SHDN!, U$10.PVDD, U$10.VCC
- new net N$2: SB2.P$2, U$1.PB12B
- new net N$25: SB1.P$2, U$1.PB12A
- new net N$26: U$2.HPOL/LOL, U$6.POS
- new net N$27: U$2.HPOR/LOR, U$8.POS
- new net N$28: SPRK1.TP, U$8.NEG
- new net N$29: R22.2, U1.PA16/PGMD4
- new net N$3: SPKR0.TP, U$6.NEG
- new net N$30: R25.1, U1.PB13/DAC0
- new net N$31: C41.1, U$9.VOUTR-
- new net N$32: C40.1, U$9.VOUTR+
- new net N$33: C41.2, R27.2
- new net N$34: C40.2, R26.2
- new net N$35: R26.1, R28.1, U$10.IN+
- new net N$36: R27.1, R29.1, U$10.IN-
- new net N$37: R28.2, U$10.FB+
- new net N$38: C39.POS, U$9.VCOM
- new net N$39: R29.2, U$10.FB-
- new net N$42: R31.1, U$9.MODE
- new net N$43: R32.1, U$9.ADR1
- new net N$44: D2.AN, R45.2
- new net N$45: D3.AN, R46.2
- new net N$46: SPK2+.TP, U$10.OUT+
- new net N$47: SPK2-.TP, U$10.OUT-
- new net N$48: D4.AN, R47.2
- new net N$49: J4.15, SB5.P$2
- new net N$52: R33.1, U$9.MS/ADR0
- new net N$53: C44.2, U$10.C1N
- new net N$54: C44.1, U$10.C1P
- new net N$7: U1.ADVREF, VREF.TP
- new net N$8: AD1.TP, U1.PA18/PGMD6/AD1
- new net PCM1789_MUTE: R30.1, U$9.AMUTEI
- new net PCM_17XX_SYSCLK: R25.2, U$2.SCKI, U$9.SCKI
- new net SW_1: R34.2, SW1.P$3, SW1.P$4, U$1.PL5C
- new net SW_2: R35.2, SW2.P$3, SW2.P$4, U$1.PL5D
- new net SW_3: R36.2, SW3.P$3, SW3.P$4, U$1.PL6A
- new net SW_4: R37.2, SW4.P$3, SW4.P$4, U$1.PL6B
- new net SW_5: R38.2, SW5.P$3, SW5.P$4, U$1.PL6C
- new net SW_6: R39.2, SW6.P$3, SW6.P$4, U$1.PL6D
- net !DISP_RESET!: now also R40.1, U1.PA8/XOUT32/PGMM0
- net +3V3: now also C35.1, C36.POS, JP1.3, R24.2, R30.2, R40.2, R41.2, R42.2, R43.2, SW1.P$1, SW1.P$2, SW2.P$1, SW2.P$2, SW3.P$1, SW3.P$2, SW4.P$1, SW4.P$2, SW5.P$1, SW5.P$2, SW6.P$1, SW6.P$2, U$1.VCCIO1@1, U$11.D, U$9.VDD
- net +5V0: now also C37.POS, C38.1, C42.1, JP1.1, U$9.VCC1, U$9.VCC2
- net DISP_CHIP_SELECT: now also U$1.PT6D; no longer U$1.PT11A
- net DISP_DB13: now also U$1.PR2B; no longer U$1.VCCIO1@1
- net DISP_DB14: now also U$1.PR2A; no longer U$1.PR2B
- net DISP_DB15: now also U$1.PT11A; no longer U$1.PR2A
- net DISP_SPI_CS: now also SB4.P$1; no longer R11.1
- net DISP_SPI_MISO: now also SB1.P$1; no longer R8.1
- net DISP_SPI_MOSI: now also SB3.P$1; no longer R10.1
- net DISP_SPI_SPCK: now also SB2.P$1; no longer R9.1
- net GND: now also C35.2, C36.NEG, C37.NEG, C38.2, C39.NEG, C42.2, C43.NEG, D2.CATH, D3.CATH, D4.CATH, R31.2, R32.2, R33.2, R34.1, R35.1, R36.1, R37.1, R38.1, R39.1, R44.1, SW7.P$1, SW7.P$2, SW8.P$3, SW8.P$4, U$10.GND, U$10.GND_PAD, U$10.PGND, U$11.COM, U$9.AGND1, U$9.AGND2, U$9.DGND
- net I2S_BCK: now also R22.1, U$9.BCK; no longer U1.PA16/PGMD4
- net I2S_DATA: now also R21.1, U$9.DIN; no longer U1.PA17/PGMD5/AD0
- net N$10: now also SB4.P$2; no longer R11.2
- net N$11: now also SB3.P$2; no longer R10.2
- net SAM4S_NRST: now also R24.1, SW7.P$3, SW7.P$4, U$9.!RST!
- net TWCK0: now also U$1.PT9C/SCL/PCLKT0_0, U$9.MC/SCL
- net TWD0: now also U$1.PT9D/SDA/PCLKC0_0, U$9.MD/SDA
- net VBUS_DETECT: now also U1.PA28
Other:
- note added: "attach speaker here"
- note added: "for speakers check out AS07108PO-3-R"
- note added: "need x7r > 6.3V"
- note added: "pcm1789 vcc1 and agnd1 caps"
- note added: "pcm1789 vcc2 and agnd2 smoothing cap"
- note added: "pcm1789 vdd and dgnd caps"
- moved on the sheet: C19, C2, C20, C21, C22, C23, C24, C3, J5, R1, R13, R14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
